Commit message: added rotatinal lidar

File: src/robot_diff_description/urdf/robot_diff.urdf (robot description, URDF)
Before this commit: robot learningrobotics, 9 links, 8 joints
Links:
- added link Cylinder, mass 0.015; collision mesh filename=package://robot_diff_description/meshes/Lidar1.stl; visual mesh filename=package://robot_diff_description/meshes/Lidar1.stl
- added link Sensor, mass 0.00008750; collision mesh filename=package://robot_diff_description/meshes/Lidar3.stl; visual mesh filename=package://robot_diff_description/meshes/Lidar3.stl
- link Lidar: mass 0.031 -> 0.016; geometry collision mesh filename=package://robot_diff_description/meshes/Lidar2.stl; visual mesh filename=package://robot_diff_description/meshes/Lidar2.stl
Joints:
- removed joint Body_to_Lidar
- added joint Body_to_Cylinder: type fixed, parent Body, child Cylinder, origin xyz=0 0.05691179 0 rpy=-1.571 -1.571 0
- added joint Cylinder_to_Lidar: type continuous, parent Cylinder, child Lidar, origin xyz=0 0 0.0263688 rpy=0 0 1.571, axis 0 0 1
- added joint Lidar_to_Sensor: type fixed, parent Lidar, child Sensor, origin xyz=0 0 0 rpy=0 0 0

Commit message: Added rotational plugin v1

File: src/robot_diff_description/urdf/robot_diff.urdf (robot description, URDF)
Before this commit: robot learningrobotics, 11 links, 10 joints
Joints:
- joint Cylinder_to_Lidar: limit (none) -> lower=-1.79769e+308 upper=1.79769e+308 effort=1.0 velocity=10.0; type continuous -> revolute
